Commit message: Bugfix: Deleted not yet existing <frame_id> tag and unused frames. Added static_transforms as workaround for not being able to use <frame_id> tag until gazebo updates to sdformat 1.12

File: src/helmoro_description/urdf/sensors/orbec_astra.urdf.xacro (robot description, xacro)
@@ -30,10 +30,4 @@
     </joint>
     <link name="camera_rgb"></link>
-    <joint name="camera_rgb_optical_joint" type="fixed">
-        <origin xyz="0 0 0" rpy="${-pi/2} 0 ${-pi/2}" />
-        <parent link="camera_rgb" />
-        <child link="camera_rgb_optical" />
-    </joint>
-    <link name="camera_rgb_optical"></link>
     <!--joints for depth_camera-->
     <joint name="camera_depth_joint" type="fixed">
@@ -43,10 +37,4 @@
     </joint>
     <link name="camera_depth"></link>
-    <joint name="camera_rgb_depth_joint" type="fixed">
-        <origin xyz="0 0 0" rpy="${-pi/2} 0 ${-pi/2}" />
-        <parent link="camera_depth" />
-        <child link="camera_depth_optical" />
-    </joint>
-    <link name="camera_depth_optical"></link>
     <!--Depth Camera Astra Pro-->
     <gazebo reference="camera_depth">
@@ -56,5 +44,5 @@
             <update_rate>30</update_rate>
             <camera>
-                <optical_frame_id>camera_depth_optical</optical_frame_id>
+                <optical_frame_id>camera_depth</optical_frame_id>
                 <horizontal_fov>1.019272</horizontal_fov> <!-- 58.4° -->
                 <image>

File: src/helmoro_description/urdf/sensors/rplidar.urdf.xacro (robot description, xacro)
@@ -24,5 +24,4 @@
         <sensor type="gpu_lidar" name="rplidar">
             <pose relative_to='${link_name}'>0 0 0 0 0 0</pose>
-            <frame_id>rplidar</frame_id>
             <update_rate>60</update_rate>
             <visualize>false</visualize>
