Commit message: Typo fixes

File: src/helmoro_description/urdf/parts/wheel.urdf.xacro (robot description, xacro)
@@ -7,5 +7,5 @@
     <xacro:property name="width"  value="0.01" />
     <xacro:property name="link_name"  value="wheel_${name}"/>
-    <xacro:property name="joint_name" value="wheel_${link_name}_joint"/>
+    <xacro:property name="joint_name" value="${link_name}_joint"/>
     <joint name="${joint_name}" type="continuous">
         <parent link="${parent_link}"/>

Commit message: fix: Add namespace to tf and tf_static topics

File: src/helmoro_description/urdf/parts/wheel.urdf.xacro (robot description, xacro)
@@ -7,5 +7,5 @@
     <xacro:property name="width"  value="0.01" />
     <xacro:property name="link_name"  value="${namespace}/wheel_${name}"/>
-    <xacro:property name="joint_name" value="${link_name}_joint"/>
+    <xacro:property name="joint_name" value="wheel_${name}_joint"/>
     <joint name="${joint_name}" type="continuous">
         <parent link="${namespace}/${parent_link}"/>

File: src/helmoro_description/urdf/plugins.urdf.xacro (robot description, xacro)
@@ -4,9 +4,12 @@
     <xacro:if value="${run_in_simulation}">
         <gazebo>
-            <plugin filename="libgz_ros2_control-system.so" name="gz_ros2_control::GazeboSimROS2ControlPlugin">
+            <plugin filename="gz_ros2_control-system" name="gz_ros2_control::GazeboSimROS2ControlPlugin">
                 <parameters>$(find helmoro_control)/config/helmoro_controller.yaml</parameters>
                 <ros>
                     <namespace>${namespace}</namespace>
                     <remapping>/robot_description:=robot_description</remapping>
+                    <remapping>/tf:=tf</remapping>
+                    <remapping>/tf_static:=tf_static</remapping>
+                    <remapping>/diagnostics:=diagnostics</remapping>
                 </ros>
             </plugin>
