Commit message: WIP: Do not use!

File: src/helmoro_description/urdf/helmoro.urdf.xacro (robot description, xacro)
@@ -11,28 +11,28 @@
     <link name="base_link"></link>
     <!-- Cover -->
-    <xacro:chassis name="chassis" gazebo="$(arg gazebo)" parent_link="base_link">
+    <xacro:chassis name="chassis" parent_link="base_link">
         <origin xyz="0 0 0.08" rpy="0 0 0"/>
     </xacro:chassis>
     <!-- Wheels -->
-    <xacro:wheel name="right_front" gazebo="$(arg gazebo)" parent_link="chassis">
+    <xacro:wheel name="right_front" run_in_simulation="$(arg run_in_simulation)" parent_link="chassis">
         <origin xyz="0.0575 0.0925 -0.035" rpy="${-pi/2} 0 0"/>
     </xacro:wheel>
-    <xacro:wheel name="left_front" gazebo="$(arg gazebo)" parent_link="chassis">
+    <xacro:wheel name="left_front" run_in_simulation="$(arg run_in_simulation)" parent_link="chassis">
         <origin xyz="0.0575 -0.0925 -0.035" rpy="${-pi/2} 0 0"/>
     </xacro:wheel>
-    <xacro:wheel name="right_back" gazebo="$(arg gazebo)" parent_link="chassis">
+    <xacro:wheel name="right_back" run_in_simulation="$(arg run_in_simulation)" parent_link="chassis">
         <origin xyz="-0.0575 0.0925 -0.035" rpy="${-pi/2} 0 0"/>
     </xacro:wheel>
-    <xacro:wheel name="left_back" gazebo="$(arg gazebo)" parent_link="chassis">
+    <xacro:wheel name="left_back" run_in_simulation="$(arg run_in_simulation)" parent_link="chassis">
         <origin xyz="-0.0575 -0.0925 -0.035" rpy="${-pi/2} 0 0"/>
     </xacro:wheel>
     <!-- Sensors -->
-    <xacro:orbec_astra name="camera" gazebo="$(arg gazebo)" parent_link="chassis">
+    <xacro:orbec_astra name="camera" parent_link="chassis">
         <origin xyz="0.114 0 0.028" rpy="0 0 0"/>
     </xacro:orbec_astra>
-    <xacro:rplidar name="lidar" gazebo="$(arg gazebo)" parent_link="chassis">
+    <xacro:rplidar name="lidar" parent_link="chassis">
         <origin xyz="0.01 0 0.0658" rpy="0 0 ${-pi/2}"/>
     </xacro:rplidar>
-    <xacro:imu name="imu" gazebo="$(arg gazebo)" parent_link="chassis">
+    <xacro:imu name="imu" parent_link="chassis">
         <origin xyz="0 0 0.001" rpy="0 0 0"/>
     </xacro:imu>

File: src/helmoro_description/urdf/parts/chassis.urdf.xacro (robot description, xacro)
@@ -1,5 +1,5 @@
 <?xml version="1.0"?>
 <robot xmlns:xacro="http://ros.org/wiki/xacro">
-<xacro:macro name="chassis" params="name gazebo parent_link *origin">
+<xacro:macro name="chassis" params="name parent_link *origin">
     <xacro:include filename="$(find helmoro_description)/urdf/utils.urdf.xacro"/>
     <xacro:property name="link_name"  value="${name}"/>

File: src/helmoro_description/urdf/parts/wheel.urdf.xacro (robot description, xacro)
@@ -1,5 +1,5 @@
 <?xml version="1.0"?>
 <robot xmlns:xacro="http://ros.org/wiki/xacro">
-<xacro:macro name="wheel" params="name gazebo parent_link *origin">
+<xacro:macro name="wheel" params="name run_in_simulation parent_link *origin">
     <xacro:include filename="$(find helmoro_description)/urdf/utils.urdf.xacro"/>
     <xacro:property name="mass"   value="0.1" />
@@ -38,8 +38,6 @@
         <minDepth>0.0001</minDepth>
         <fdir1>1 0 0</fdir1>
-        <slip1>0.5</slip1>
-        <slip2>0</slip2>
     </gazebo>
-    <xacro:if value="${gazebo == 'false'}">
+    <xacro:if value="${run_in_simulation == 'false'}">
         <ros2_control name="${link_name}_controller" type="system">
         <hardware>
@@ -53,8 +51,8 @@
         </ros2_control>
     </xacro:if>
-    <xacro:if value="${gazebo == 'true'}">
+    <xacro:if value="${run_in_simulation == 'true'}">
         <ros2_control name="${link_name}_controller" type="system">
         <hardware>
-            <plugin>ign_ros2_control/IgnitionSystem</plugin>
+            <plugin>gazebo_ros2_control/GazeboSystem</plugin>
         </hardware>
         <joint name="${joint_name}">

File: src/helmoro_description/urdf/sensors/imu.urdf.xacro (robot description, xacro)
@@ -1,5 +1,5 @@
 <?xml version="1.0"?>
 <robot xmlns:xacro="http://ros.org/wiki/xacro">
-<xacro:macro name="imu" params="name gazebo parent_link *origin">
+<xacro:macro name="imu" params="name parent_link *origin">
     <xacro:include filename="$(find helmoro_description)/urdf/utils.urdf.xacro"/>
     <xacro:property name="joint_name" value="${name}_joint"/>
@@ -14,5 +14,5 @@
         <gravity>true</gravity>
         <sensor name="imu_sensor" type="imu">
-            <ignition_frame_id>${link_name}</ignition_frame_id>
+            <pose relative_to='${link_name}'>0 0 0 0 0 0</pose>
             <always_on>true</always_on>
             <update_rate>100</update_rate>
@@ -22,4 +22,7 @@
         </sensor>
     </gazebo>
+    <plugin filename="gz-sim-imu-system"
+        name="gz::sim::systems::Imu">
+    </plugin>
 </xacro:macro>
 </robot>

File: src/helmoro_description/urdf/sensors/orbec_astra.urdf.xacro (robot description, xacro)
@@ -1,5 +1,5 @@
 <?xml version="1.0"?>
 <robot xmlns:xacro="http://ros.org/wiki/xacro">
-<xacro:macro name="orbec_astra" params="name gazebo parent_link *origin">
+<xacro:macro name="orbec_astra" params="name parent_link *origin">
     <xacro:include filename="$(find helmoro_description)/urdf/utils.urdf.xacro"/>
     <xacro:property name="camera_joint_name" value="${name}_joint"/>
@@ -52,11 +52,10 @@
     <gazebo reference="camera_depth">
         <sensor name="depth_camera" type="depth_camera">
+        <pose relative_to='camera_depth'>0 0 0 0 0 0</pose>
         <always_on>0</always_on>
         <update_rate>30</update_rate>
         <topic>depth_camera</topic>
-        <ignition_frame_id>camera_depth</ignition_frame_id>
         <camera>
             <horizontal_fov>1.019272</horizontal_fov> <!-- 58.4° -->
-            <vertical_fov>0.7941248</vertical_fov> <!-- 45.5° -->
             <image>
                 <width>640</width>
@@ -74,11 +73,10 @@
     <gazebo reference="camera_rgb">
         <sensor name="rgb_camera" type="camera">
+        <pose relative_to='camera_rgb'>0 0 0 0 0 0</pose>
         <always_on>0</always_on>
         <update_rate>30</update_rate>
         <topic>rgb_camera</topic>
-        <ignition_frame_id>camera_rgb</ignition_frame_id>
         <camera>
             <horizontal_fov>1.101303</horizontal_fov> <!-- 63.1° -->
-            <vertical_fov>0.8621927</vertical_fov> <!-- 49.4° -->
             <image>
                 <width>640</width>

File: src/helmoro_description/urdf/sensors/rplidar.urdf.xacro (robot description, xacro)
@@ -1,5 +1,5 @@
 <?xml version="1.0"?>
 <robot xmlns:xacro="http://ros.org/wiki/xacro">
-<xacro:macro name="rplidar" params="name gazebo parent_link *origin">
+<xacro:macro name="rplidar" params="name parent_link *origin">
     <xacro:include filename="$(find helmoro_description)/urdf/utils.urdf.xacro"/>
     <xacro:property name="joint_name" value="${name}_joint"/>
@@ -27,5 +27,4 @@
         <update_rate>60</update_rate>
         <visualize>false</visualize>
-        <ignition_frame_id>${name}</ignition_frame_id>
         <ray>
             <scan>
@@ -54,4 +53,9 @@
         </sensor>
     </gazebo>
+    <plugin
+        filename="gz-sim-sensors-system"
+        name="gz::sim::systems::Sensors">
+        <render_engine>ogre2</render_engine>
+    </plugin>
 </xacro:macro>
 </robot>

Commit message: Added namespaces to urdf

File: src/helmoro_description/urdf/helmoro.urdf.xacro (robot description, xacro)
@@ -2,4 +2,5 @@
 <robot name="321" xmlns:xacro="http://ros.org/wiki/xacro">
     <xacro:arg name="namespace" default="123" />
+    <xacro:arg name="run_in_simulation" default="false" />
     <xacro:include filename="$(find helmoro_description)/urdf/utils.urdf.xacro"/>
     <xacro:include filename="$(find helmoro_description)/urdf/parts/chassis.urdf.xacro"/>
@@ -11,28 +12,28 @@
     <link name="base_link"></link>
     <!-- Cover -->
-    <xacro:chassis name="chassis" gazebo="$(arg gazebo)" parent_link="base_link">
+    <xacro:chassis name="chassis" namespace="$(arg namespace)" parent_link="base_link">
         <origin xyz="0 0 0.08" rpy="0 0 0"/>
     </xacro:chassis>
     <!-- Wheels -->
-    <xacro:wheel name="right_front" gazebo="$(arg gazebo)" parent_link="chassis">
+    <xacro:wheel name="right_front" namespace="$(arg namespace)" run_in_simulation="$(arg run_in_simulation)" parent_link="chassis">
         <origin xyz="0.0575 0.0925 -0.035" rpy="${-pi/2} 0 0"/>
     </xacro:wheel>
-    <xacro:wheel name="left_front" gazebo="$(arg gazebo)" parent_link="chassis">
+    <xacro:wheel name="left_front" namespace="$(arg namespace)" run_in_simulation="$(arg run_in_simulation)" parent_link="chassis">
         <origin xyz="0.0575 -0.0925 -0.035" rpy="${-pi/2} 0 0"/>
     </xacro:wheel>
-    <xacro:wheel name="right_back" gazebo="$(arg gazebo)" parent_link="chassis">
+    <xacro:wheel name="right_back" namespace="$(arg namespace)" run_in_simulation="$(arg run_in_simulation)" parent_link="chassis">
         <origin xyz="-0.0575 0.0925 -0.035" rpy="${-pi/2} 0 0"/>
     </xacro:wheel>
-    <xacro:wheel name="left_back" gazebo="$(arg gazebo)" parent_link="chassis">
+    <xacro:wheel name="left_back" namespace="$(arg namespace)" run_in_simulation="$(arg run_in_simulation)" parent_link="chassis">
         <origin xyz="-0.0575 -0.0925 -0.035" rpy="${-pi/2} 0 0"/>
     </xacro:wheel>
     <!-- Sensors -->
-    <xacro:orbec_astra name="camera" gazebo="$(arg gazebo)" parent_link="chassis">
+    <xacro:orbec_astra name="camera" namespace="$(arg namespace)" parent_link="chassis">
         <origin xyz="0.114 0 0.028" rpy="0 0 0"/>
     </xacro:orbec_astra>
-    <xacro:rplidar name="lidar" gazebo="$(arg gazebo)" parent_link="chassis">
+    <xacro:rplidar name="lidar" namespace="$(arg namespace)" parent_link="chassis">
         <origin xyz="0.01 0 0.0658" rpy="0 0 ${-pi/2}"/>
     </xacro:rplidar>
-    <xacro:imu name="imu" gazebo="$(arg gazebo)" parent_link="chassis">
+    <xacro:imu name="imu" namespace="$(arg namespace)" parent_link="chassis">
         <origin xyz="0 0 0.001" rpy="0 0 0"/>
     </xacro:imu>

File: src/helmoro_description/urdf/parts/chassis.urdf.xacro (robot description, xacro)
@@ -1,5 +1,5 @@
 <?xml version="1.0"?>
 <robot xmlns:xacro="http://ros.org/wiki/xacro">
-<xacro:macro name="chassis" params="name gazebo parent_link *origin">
+<xacro:macro name="chassis" params="name namespace parent_link *origin">
     <xacro:include filename="$(find helmoro_description)/urdf/utils.urdf.xacro"/>
     <xacro:property name="link_name"  value="${name}"/>

File: src/helmoro_description/urdf/parts/wheel.urdf.xacro (robot description, xacro)
@@ -1,5 +1,5 @@
 <?xml version="1.0"?>
 <robot xmlns:xacro="http://ros.org/wiki/xacro">
-<xacro:macro name="wheel" params="name gazebo parent_link *origin">
+<xacro:macro name="wheel" params="name namespace run_in_simulation parent_link *origin">
     <xacro:include filename="$(find helmoro_description)/urdf/utils.urdf.xacro"/>
     <xacro:property name="mass"   value="0.1" />
@@ -16,11 +16,11 @@
     <link name="${link_name}">
         <visual>
-        <geometry>
-            <cylinder length="${width}" radius="${radius}"/>
-        </geometry>
-        <!-- Give black color to wheels in Rviz -->
-        <material name="HELMORO_BLACK">
-            <color rgba="0.0 0.0 0.0 1.0"/>
-        </material>
+            <geometry>
+                <cylinder length="${width}" radius="${radius}"/>
+            </geometry>
+            <!-- Give black color to wheels in Rviz -->
+            <material name="HELMORO_BLACK">
+                <color rgba="0.0 0.0 0.0 1.0"/>
+            </material>
         </visual>
         <collision>
@@ -38,8 +38,6 @@
         <minDepth>0.0001</minDepth>
         <fdir1>1 0 0</fdir1>
-        <slip1>0.5</slip1>
-        <slip2>0</slip2>
     </gazebo>
-    <xacro:if value="${gazebo == 'false'}">
+    <xacro:if value="${run_in_simulation == 'false'}">
         <ros2_control name="${link_name}_controller" type="system">
         <hardware>
@@ -53,8 +51,8 @@
         </ros2_control>
     </xacro:if>
-    <xacro:if value="${gazebo == 'true'}">
+    <xacro:if value="${run_in_simulation == 'true'}">
         <ros2_control name="${link_name}_controller" type="system">
         <hardware>
-            <plugin>ign_ros2_control/IgnitionSystem</plugin>
+            <plugin>gazebo_ros2_control/GazeboSystem</plugin>
         </hardware>
         <joint name="${joint_name}">

File: src/helmoro_description/urdf/sensors/imu.urdf.xacro (robot description, xacro)
@@ -1,5 +1,5 @@
 <?xml version="1.0"?>
 <robot xmlns:xacro="http://ros.org/wiki/xacro">
-<xacro:macro name="imu" params="name gazebo parent_link *origin">
+<xacro:macro name="imu" params="name namespace parent_link *origin">
     <xacro:include filename="$(find helmoro_description)/urdf/utils.urdf.xacro"/>
     <xacro:property name="joint_name" value="${name}_joint"/>
@@ -14,9 +14,8 @@
         <gravity>true</gravity>
         <sensor name="imu_sensor" type="imu">
-            <ignition_frame_id>${link_name}</ignition_frame_id>
+            <pose relative_to='${link_name}'>0 0 0 0 0 0</pose>
             <always_on>true</always_on>
             <update_rate>100</update_rate>
             <visualize>true</visualize>
-            <topic>imu</topic>
             <pose>0 0 0 0 0 0</pose>
         </sensor>

File: src/helmoro_description/urdf/sensors/orbec_astra.urdf.xacro (robot description, xacro)
@@ -1,5 +1,5 @@
 <?xml version="1.0"?>
 <robot xmlns:xacro="http://ros.org/wiki/xacro">
-<xacro:macro name="orbec_astra" params="name gazebo parent_link *origin">
+<xacro:macro name="orbec_astra" params="name namespace parent_link *origin">
     <xacro:include filename="$(find helmoro_description)/urdf/utils.urdf.xacro"/>
     <xacro:property name="camera_joint_name" value="${name}_joint"/>
@@ -52,21 +52,20 @@
     <gazebo reference="camera_depth">
         <sensor name="depth_camera" type="depth_camera">
-        <always_on>0</always_on>
-        <update_rate>30</update_rate>
-        <topic>depth_camera</topic>
-        <ignition_frame_id>camera_depth</ignition_frame_id>
-        <camera>
-            <horizontal_fov>1.019272</horizontal_fov> <!-- 58.4° -->
-            <vertical_fov>0.7941248</vertical_fov> <!-- 45.5° -->
-            <image>
-                <width>640</width>
-                <height>480</height>
-                <format>R8G8B8</format>
-            </image>
-            <clip>
-                <near>0.1</near>
-                <far>100.0</far>
-            </clip>
-        </camera>
+            <pose relative_to='camera_depth'>0 0 0 0 0 0</pose>
+            <always_on>0</always_on>
+            <update_rate>30</update_rate>
+            <camera>
+                <optical_frame_id>camera_depth_optical</optical_frame_id>
+                <horizontal_fov>1.019272</horizontal_fov> <!-- 58.4° -->
+                <image>
+                    <width>640</width>
+                    <height>480</height>
+                    <format>R8G8B8</format>
+                </image>
+                <clip>
+                    <near>0.1</near>
+                    <far>100.0</far>
+                </clip>
+            </camera>
         </sensor>
     </gazebo>
@@ -74,21 +73,20 @@
     <gazebo reference="camera_rgb">
         <sensor name="rgb_camera" type="camera">
-        <always_on>0</always_on>
-        <update_rate>30</update_rate>
-        <topic>rgb_camera</topic>
-        <ignition_frame_id>camera_rgb</ignition_frame_id>
-        <camera>
-            <horizontal_fov>1.101303</horizontal_fov> <!-- 63.1° -->
-            <vertical_fov>0.8621927</vertical_fov> <!-- 49.4° -->
-            <image>
-                <width>640</width>
-                <height>480</height>
-                <format>R8G8B8</format>
-            </image>
-            <clip>
-                <near>0.1</near>
-                <far>100.0</far>
-            </clip>
-        </camera>
+            <pose relative_to='camera_rgb'>0 0 0 0 0 0</pose>
+            <always_on>0</always_on>
+            <update_rate>30</update_rate>
+            <camera>
+                <optical_frame_id>camera_rgb_optical</optical_frame_id>
+                <horizontal_fov>1.101303</horizontal_fov> <!-- 63.1° -->
+                <image>
+                    <width>640</width>
+                    <height>480</height>
+                    <format>R8G8B8</format>
+                </image>
+                <clip>
+                    <near>0.1</near>
+                    <far>100.0</far>
+                </clip>
+            </camera>
         </sensor>
     </gazebo>

File: src/helmoro_description/urdf/sensors/rplidar.urdf.xacro (robot description, xacro)
@@ -1,5 +1,5 @@
-<?xml version="1.0"?>
+<?xml version="1.1"?>
 <robot xmlns:xacro="http://ros.org/wiki/xacro">
-<xacro:macro name="rplidar" params="name gazebo parent_link *origin">
+<xacro:macro name="rplidar" params="name namespace parent_link *origin">
     <xacro:include filename="$(find helmoro_description)/urdf/utils.urdf.xacro"/>
     <xacro:property name="joint_name" value="${name}_joint"/>
@@ -23,33 +23,32 @@
     <gazebo reference="${link_name}">
         <sensor type="gpu_lidar" name="rplidar">
-        <pose relative_to='${link_name}'>0 0 0 0 0 0</pose>
-        <topic>scan</topic>
-        <update_rate>60</update_rate>
-        <visualize>false</visualize>
-        <ignition_frame_id>${name}</ignition_frame_id>
-        <ray>
-            <scan>
-            <horizontal>
-                <samples>720</samples>
-                <resolution>1</resolution>
-                <min_angle>0</min_angle> <!--0 degrees-->
-                <max_angle>${2*pi}</max_angle> <!--360 degrees-->
-            </horizontal>
-            </scan>
-            <range>
-            <min>0.15</min> <!--should be 0.15-->
-            <max>12.0</max>
-            <resolution>0.01</resolution>
-            </range>
-            <noise>
-            <type>gaussian</type>
-            <!-- Noise parameters based on published spec for Hokuyo laser
-                achieving "+-30mm" accuracy at range < 10m.  A mean of 0.0m and
-                stddev of 0.01m will put 99.7% of samples within 0.03m of the true
-                reading. -->
-            <mean>0.0</mean>
-            <stddev>0.01</stddev>
-            </noise>
-        </ray>
+            <pose relative_to='${link_name}'>0 0 0 0 0 0</pose>
+            <frame_id>rplidar</frame_id>
+            <update_rate>60</update_rate>
+            <visualize>false</visualize>
+            <lidar>
+                <scan>
+                    <horizontal>
+                        <samples>720</samples>
+                        <resolution>1</resolution>
+                        <min_angle>0</min_angle> <!--0 degrees-->
+                        <max_angle>${2*pi}</max_angle> <!--360 degrees-->
+                    </horizontal>
+                </scan>
+                <range>
+                    <min>0.15</min> <!--should be 0.15-->
+                    <max>12.0</max>
+                    <resolution>0.01</resolution>
+                </range>
+                <noise>
+                    <type>gaussian</type>
+                    <!-- Noise parameters based on published spec for Hokuyo laser
+                        achieving "+-30mm" accuracy at range < 10m.  A mean of 0.0m and
+                        stddev of 0.01m will put 99.7% of samples within 0.03m of the true
+                        reading. -->
+                    <mean>0.0</mean>
+                    <stddev>0.01</stddev>
+                </noise>
+            </lidar>
         </sensor>
     </gazebo>
