Commit message: Added control pkg

File: src/helmoro_description/urdf/helmoro.urdf.xacro (robot description, xacro)
@@ -1,6 +1,7 @@
 <?xml version="1.0" ?>
-<robot name="321" xmlns:xacro="http://ros.org/wiki/xacro">
+<robot name="example_robot_name" xmlns:xacro="http://ros.org/wiki/xacro">
     <xacro:arg name="namespace" default="123" />
     <xacro:arg name="run_in_simulation" default="false" />
+    <xacro:include filename="$(find helmoro_description)/urdf/plugins.urdf.xacro"/>
     <xacro:include filename="$(find helmoro_description)/urdf/utils.urdf.xacro"/>
     <xacro:include filename="$(find helmoro_description)/urdf/parts/chassis.urdf.xacro"/>
@@ -16,14 +17,14 @@
     </xacro:chassis>
     <!-- Wheels -->
-    <xacro:wheel name="right_front" namespace="$(arg namespace)" run_in_simulation="$(arg run_in_simulation)" parent_link="chassis">
+    <xacro:wheel name="left_front" namespace="$(arg namespace)" run_in_simulation="$(arg run_in_simulation)" parent_link="chassis">
         <origin xyz="0.0575 0.0925 -0.035" rpy="${-pi/2} 0 0"/>
     </xacro:wheel>
-    <xacro:wheel name="left_front" namespace="$(arg namespace)" run_in_simulation="$(arg run_in_simulation)" parent_link="chassis">
+    <xacro:wheel name="right_front" namespace="$(arg namespace)" run_in_simulation="$(arg run_in_simulation)" parent_link="chassis">
         <origin xyz="0.0575 -0.0925 -0.035" rpy="${-pi/2} 0 0"/>
     </xacro:wheel>
-    <xacro:wheel name="right_back" namespace="$(arg namespace)" run_in_simulation="$(arg run_in_simulation)" parent_link="chassis">
+    <xacro:wheel name="left_back" namespace="$(arg namespace)" run_in_simulation="$(arg run_in_simulation)" parent_link="chassis">
         <origin xyz="-0.0575 0.0925 -0.035" rpy="${-pi/2} 0 0"/>
     </xacro:wheel>
-    <xacro:wheel name="left_back" namespace="$(arg namespace)" run_in_simulation="$(arg run_in_simulation)" parent_link="chassis">
+    <xacro:wheel name="right_back" namespace="$(arg namespace)" run_in_simulation="$(arg run_in_simulation)" parent_link="chassis">
         <origin xyz="-0.0575 -0.0925 -0.035" rpy="${-pi/2} 0 0"/>
     </xacro:wheel>
@@ -38,14 +39,5 @@
         <origin xyz="0 0 0.001" rpy="0 0 0"/>
     </xacro:imu>
-    <!-- TODO: Control -->
-    <!-- <xacro:if value="${'$(arg gazebo)' == 'true'}">
-        <gazebo>
-            <plugin filename="gz_ros2_control-system" name="gz_ros2_control::GazeboSimROS2ControlPlugin">
-                <parameters>$(find helmoro_control)/config/helmoro_controller.yaml</parameters>
-                <ros>
-                <namespace>$(arg namespace)</namespace>
-                </ros>
-            </plugin>
-        </gazebo>
-    </xacro:if> -->
+    <!-- Plugins -->
+    <xacro:control namespace="$(arg namespace)" run_in_simulation="$(arg run_in_simulation)"></xacro:control>
 </robot>

File: src/helmoro_description/urdf/parts/wheel.urdf.xacro (robot description, xacro)
@@ -39,26 +39,26 @@
         <fdir1>1 0 0</fdir1>
     </gazebo>
-    <xacro:if value="${run_in_simulation == 'false'}">
+    <xacro:unless value="${run_in_simulation}">
         <ros2_control name="${link_name}_controller" type="system">
-        <hardware>
-            <plugin>fake_components/GenericSystem</plugin>
-        </hardware>
-        <joint name="${joint_name}">
-            <state_interface name="velocity" />
-            <state_interface name="position" />
-            <command_interface name="velocity" />
-        </joint>
+            <hardware>
+                <plugin>diff_drive/HelmoroSystem</plugin>
+            </hardware>
+            <joint name="${joint_name}">
+                <state_interface name="velocity" />
+                <state_interface name="position" />
+                <command_interface name="velocity" />
+            </joint>
         </ros2_control>
-    </xacro:if>
-    <xacro:if value="${run_in_simulation == 'true'}">
+    </xacro:unless>
+    <xacro:if value="${run_in_simulation}">
         <ros2_control name="${link_name}_controller" type="system">
-        <hardware>
-            <plugin>gazebo_ros2_control/GazeboSystem</plugin>
-        </hardware>
-        <joint name="${joint_name}">
-            <state_interface name="velocity" />
-            <state_interface name="position" />
-            <command_interface name="velocity" />
-        </joint>
+            <hardware>
+                <plugin>gz_ros2_control/GazeboSimSystem</plugin>
+            </hardware>
+            <joint name="${joint_name}">
+                <state_interface name="velocity" />
+                <state_interface name="position" />
+                <command_interface name="velocity" />
+            </joint>
         </ros2_control>
     </xacro:if>

Commit message: Cleaned up control configs and adjusted namespaces to follow standard

File: src/helmoro_description/urdf/helmoro.urdf.xacro (robot description, xacro)
@@ -11,5 +11,5 @@
     <xacro:include filename="$(find helmoro_description)/urdf/sensors/imu.urdf.xacro"/>
     <!-- Base Link -->
-    <link name="base_link"></link>
+    <link name="$(arg namespace)/base_link"></link>
     <!-- Cover -->
     <xacro:chassis name="chassis" namespace="$(arg namespace)" parent_link="base_link">

File: src/helmoro_description/urdf/parts/chassis.urdf.xacro (robot description, xacro)
@@ -3,8 +3,8 @@
 <xacro:macro name="chassis" params="name namespace parent_link *origin">
     <xacro:include filename="$(find helmoro_description)/urdf/utils.urdf.xacro"/>
-    <xacro:property name="link_name"  value="${name}"/>
+    <xacro:property name="link_name"  value="${namespace}/${name}"/>
     <xacro:property name="joint_name" value="${link_name}_joint"/>
     <joint name="${joint_name}" type="fixed">
-        <parent link="${parent_link}"/>
+        <parent link="${namespace}/${parent_link}"/>
         <child link="${link_name}"/>
         <xacro:insert_block name="origin"/>

File: src/helmoro_description/urdf/parts/wheel.urdf.xacro (robot description, xacro)
@@ -6,8 +6,8 @@
     <xacro:property name="radius" value="0.045" />
     <xacro:property name="width"  value="0.01" />
-    <xacro:property name="link_name"  value="wheel_${name}"/>
+    <xacro:property name="link_name"  value="${namespace}/wheel_${name}"/>
     <xacro:property name="joint_name" value="${link_name}_joint"/>
     <joint name="${joint_name}" type="continuous">
-        <parent link="${parent_link}"/>
+        <parent link="${namespace}/${parent_link}"/>
         <child link="${link_name}"/>
         <xacro:insert_block name="origin"/>

File: src/helmoro_description/urdf/sensors/imu.urdf.xacro (robot description, xacro)
@@ -3,8 +3,8 @@
 <xacro:macro name="imu" params="name namespace parent_link *origin">
     <xacro:include filename="$(find helmoro_description)/urdf/utils.urdf.xacro"/>
-    <xacro:property name="joint_name" value="${name}_joint"/>
-    <xacro:property name="link_name" value="${name}"/>
+    <xacro:property name="link_name" value="${namespace}/${name}"/>
+    <xacro:property name="joint_name" value="${link_name}_joint"/>
     <joint name="${joint_name}" type="fixed">
-        <parent link="${parent_link}"/>
+        <parent link="${namespace}/${parent_link}"/>
         <child link="${link_name}"/>
         <xacro:insert_block name="origin"/>

File: src/helmoro_description/urdf/sensors/orbec_astra.urdf.xacro (robot description, xacro)
@@ -3,9 +3,9 @@
 <xacro:macro name="orbec_astra" params="name namespace parent_link *origin">
     <xacro:include filename="$(find helmoro_description)/urdf/utils.urdf.xacro"/>
-    <xacro:property name="camera_joint_name" value="${name}_joint"/>
-    <xacro:property name="link_name" value="${name}_mesh"/>
+    <xacro:property name="link_name" value="${namespace}/${name}_mesh"/>
+    <xacro:property name="camera_joint_name" value="${namespace}/${name}_joint"/>
     <!-- joint for camera mesh -->
     <joint name="${camera_joint_name}" type="fixed">
-        <parent link="${parent_link}"/>
+        <parent link="${namespace}/${parent_link}"/>
         <child link="${link_name}"/>
         <xacro:insert_block name="origin"/>
@@ -27,22 +27,22 @@
         <origin xyz="0 0.045 0" rpy="0 0 0" />
         <parent link="${link_name}" />
-        <child link="camera_rgb" />
+        <child link="${namespace}/camera_rgb" />
     </joint>
-    <link name="camera_rgb"></link>
+    <link name="${namespace}/camera_rgb"></link>
     <!--joints for depth_camera-->
     <joint name="camera_depth_joint" type="fixed">
         <origin xyz="0 0.02 0" rpy="0 0 0" />
         <parent link="${link_name}" />
-        <child link="camera_depth" />
+        <child link="${namespace}/camera_depth" />
     </joint>
-    <link name="camera_depth"></link>
+    <link name="${namespace}/camera_depth"></link>
     <!--Depth Camera Astra Pro-->
-    <gazebo reference="camera_depth">
+    <gazebo reference="${namespace}/camera_depth">
         <sensor name="depth_camera" type="depth_camera">
-            <pose relative_to='camera_depth'>0 0 0 0 0 0</pose>
+            <pose relative_to='${namespace}/camera_depth'>0 0 0 0 0 0</pose>
             <always_on>0</always_on>
             <update_rate>30</update_rate>
             <camera>
-                <optical_frame_id>camera_depth</optical_frame_id>
+                <optical_frame_id>${namespace}/camera_depth</optical_frame_id>
                 <horizontal_fov>1.019272</horizontal_fov> <!-- 58.4° -->
                 <image>
@@ -59,11 +59,11 @@
     </gazebo>
     <!--RGB Camera Astra Pro-->
-    <gazebo reference="camera_rgb">
+    <gazebo reference="${namespace}/camera_rgb">
         <sensor name="rgb_camera" type="camera">
-            <pose relative_to='camera_rgb'>0 0 0 0 0 0</pose>
+            <pose relative_to='${namespace}/camera_rgb'>0 0 0 0 0 0</pose>
             <always_on>0</always_on>
             <update_rate>30</update_rate>
             <camera>
-                <optical_frame_id>camera_rgb_optical</optical_frame_id>
+                <optical_frame_id>${namespace}/camera_rgb</optical_frame_id>
                 <horizontal_fov>1.101303</horizontal_fov> <!-- 63.1° -->
                 <image>

File: src/helmoro_description/urdf/sensors/rplidar.urdf.xacro (robot description, xacro)
@@ -3,8 +3,8 @@
 <xacro:macro name="rplidar" params="name namespace parent_link *origin">
     <xacro:include filename="$(find helmoro_description)/urdf/utils.urdf.xacro"/>
-    <xacro:property name="joint_name" value="${name}_joint"/>
-    <xacro:property name="link_name" value="${name}"/>
+    <xacro:property name="joint_name" value="${namespace}/${name}_joint"/>
+    <xacro:property name="link_name" value="${namespace}/${name}"/>
     <joint name="${joint_name}" type="fixed">
-        <parent link="${parent_link}"/>
+        <parent link="${namespace}/${parent_link}"/>
         <child link="${link_name}"/>
         <xacro:insert_block name="origin"/>

Commit message: refactor: removed dependency on fixed namespaces

File: src/helmoro_description/urdf/helmoro.urdf.xacro (robot description, xacro)
@@ -11,30 +11,30 @@
     <xacro:include filename="$(find helmoro_description)/urdf/sensors/imu.urdf.xacro"/>
     <!-- Base Link -->
-    <link name="$(arg namespace)/base_link"></link>
+    <link name="base_link"></link>
     <!-- Cover -->
-    <xacro:chassis name="chassis" namespace="$(arg namespace)" parent_link="base_link">
+    <xacro:chassis name="chassis" parent_link="base_link">
         <origin xyz="0 0 0.08" rpy="0 0 0"/>
     </xacro:chassis>
     <!-- Wheels -->
-    <xacro:wheel name="left_front" namespace="$(arg namespace)" run_in_simulation="$(arg run_in_simulation)" parent_link="chassis">
+    <xacro:wheel name="left_front" run_in_simulation="$(arg run_in_simulation)" parent_link="chassis">
         <origin xyz="0.0575 0.0925 -0.035" rpy="${-pi/2} 0 0"/>
     </xacro:wheel>
-    <xacro:wheel name="right_front" namespace="$(arg namespace)" run_in_simulation="$(arg run_in_simulation)" parent_link="chassis">
+    <xacro:wheel name="right_front" run_in_simulation="$(arg run_in_simulation)" parent_link="chassis">
         <origin xyz="0.0575 -0.0925 -0.035" rpy="${-pi/2} 0 0"/>
     </xacro:wheel>
-    <xacro:wheel name="left_back" namespace="$(arg namespace)" run_in_simulation="$(arg run_in_simulation)" parent_link="chassis">
+    <xacro:wheel name="left_back" run_in_simulation="$(arg run_in_simulation)" parent_link="chassis">
         <origin xyz="-0.0575 0.0925 -0.035" rpy="${-pi/2} 0 0"/>
     </xacro:wheel>
-    <xacro:wheel name="right_back" namespace="$(arg namespace)" run_in_simulation="$(arg run_in_simulation)" parent_link="chassis">
+    <xacro:wheel name="right_back" run_in_simulation="$(arg run_in_simulation)" parent_link="chassis">
         <origin xyz="-0.0575 -0.0925 -0.035" rpy="${-pi/2} 0 0"/>
     </xacro:wheel>
     <!-- Sensors -->
-    <xacro:orbec_astra name="camera" namespace="$(arg namespace)" parent_link="chassis">
+    <xacro:orbec_astra name="camera" parent_link="chassis">
         <origin xyz="0.114 0 0.028" rpy="0 0 0"/>
     </xacro:orbec_astra>
-    <xacro:rplidar name="lidar" namespace="$(arg namespace)" parent_link="chassis">
+    <xacro:rplidar name="lidar" parent_link="chassis">
         <origin xyz="0.01 0 0.0658" rpy="0 0 ${-pi/2}"/>
     </xacro:rplidar>
-    <xacro:imu name="imu" namespace="$(arg namespace)" parent_link="chassis">
+    <xacro:imu name="imu" parent_link="chassis">
         <origin xyz="0 0 0.001" rpy="0 0 0"/>
     </xacro:imu>

File: src/helmoro_description/urdf/parts/chassis.urdf.xacro (robot description, xacro)
@@ -1,10 +1,10 @@
 <?xml version="1.0"?>
 <robot xmlns:xacro="http://ros.org/wiki/xacro">
-<xacro:macro name="chassis" params="name namespace parent_link *origin">
+<xacro:macro name="chassis" params="name parent_link *origin">
     <xacro:include filename="$(find helmoro_description)/urdf/utils.urdf.xacro"/>
-    <xacro:property name="link_name"  value="${namespace}/${name}"/>
+    <xacro:property name="link_name"  value="${name}"/>
     <xacro:property name="joint_name" value="${link_name}_joint"/>
     <joint name="${joint_name}" type="fixed">
-        <parent link="${namespace}/${parent_link}"/>
+        <parent link="${parent_link}"/>
         <child link="${link_name}"/>
         <xacro:insert_block name="origin"/>

File: src/helmoro_description/urdf/parts/wheel.urdf.xacro (robot description, xacro)
@@ -1,13 +1,13 @@
 <?xml version="1.0"?>
 <robot xmlns:xacro="http://ros.org/wiki/xacro">
-<xacro:macro name="wheel" params="name namespace run_in_simulation parent_link *origin">
+<xacro:macro name="wheel" params="name run_in_simulation parent_link *origin">
     <xacro:include filename="$(find helmoro_description)/urdf/utils.urdf.xacro"/>
     <xacro:property name="mass"   value="0.1" />
     <xacro:property name="radius" value="0.045" />
     <xacro:property name="width"  value="0.01" />
-    <xacro:property name="link_name"  value="${namespace}/wheel_${name}"/>
+    <xacro:property name="link_name"  value="wheel_${name}"/>
     <xacro:property name="joint_name" value="wheel_${name}_joint"/>
     <joint name="${joint_name}" type="continuous">
-        <parent link="${namespace}/${parent_link}"/>
+        <parent link="${parent_link}"/>
         <child link="${link_name}"/>
         <xacro:insert_block name="origin"/>

File: src/helmoro_description/urdf/sensors/imu.urdf.xacro (robot description, xacro)
@@ -1,10 +1,10 @@
 <?xml version="1.0"?>
 <robot xmlns:xacro="http://ros.org/wiki/xacro">
-<xacro:macro name="imu" params="name namespace parent_link *origin">
+<xacro:macro name="imu" params="name parent_link *origin">
     <xacro:include filename="$(find helmoro_description)/urdf/utils.urdf.xacro"/>
-    <xacro:property name="link_name" value="${namespace}/${name}"/>
+    <xacro:property name="link_name" value="${name}"/>
     <xacro:property name="joint_name" value="${link_name}_joint"/>
     <joint name="${joint_name}" type="fixed">
-        <parent link="${namespace}/${parent_link}"/>
+        <parent link="${parent_link}"/>
         <child link="${link_name}"/>
         <xacro:insert_block name="origin"/>
@@ -68,12 +68,4 @@
             </linear_acceleration>
         </imu>
-        <!-- <xacro:if value="${gazebo == 'classic'}">
-            <plugin name="${name}_plugin" filename="libgazebo_ros_create_imu.so">
-            <ros>
-                <namespace>${namespace}</namespace>
-                <remapping>~/out:=imu</remapping>
-            </ros>
-            </plugin>
-        </xacro:if> -->
         </sensor>
     </gazebo>

File: src/helmoro_description/urdf/sensors/orbec_astra.urdf.xacro (robot description, xacro)
@@ -1,11 +1,11 @@
 <?xml version="1.0"?>
 <robot xmlns:xacro="http://ros.org/wiki/xacro">
-<xacro:macro name="orbec_astra" params="name namespace parent_link *origin">
+<xacro:macro name="orbec_astra" params="name parent_link *origin">
     <xacro:include filename="$(find helmoro_description)/urdf/utils.urdf.xacro"/>
-    <xacro:property name="link_name" value="${namespace}/${name}_mesh"/>
-    <xacro:property name="camera_joint_name" value="${namespace}/${name}_joint"/>
+    <xacro:property name="link_name" value="${name}_mesh"/>
+    <xacro:property name="camera_joint_name" value="${name}_joint"/>
     <!-- joint for camera mesh -->
     <joint name="${camera_joint_name}" type="fixed">
-        <parent link="${namespace}/${parent_link}"/>
+        <parent link="${parent_link}"/>
         <child link="${link_name}"/>
         <xacro:insert_block name="origin"/>
@@ -27,22 +27,22 @@
         <origin xyz="0 0.045 0" rpy="0 0 0" />
         <parent link="${link_name}" />
-        <child link="${namespace}/camera_rgb" />
+        <child link="camera_rgb" />
     </joint>
-    <link name="${namespace}/camera_rgb"></link>
+    <link name="camera_rgb"></link>
     <!--joints for depth_camera-->
     <joint name="camera_depth_joint" type="fixed">
         <origin xyz="0 0.02 0" rpy="0 0 0" />
         <parent link="${link_name}" />
-        <child link="${namespace}/camera_depth" />
+        <child link="camera_depth" />
     </joint>
-    <link name="${namespace}/camera_depth"></link>
+    <link name="camera_depth"></link>
     <!--Depth Camera Astra Pro-->
-    <gazebo reference="${namespace}/camera_depth">
+    <gazebo reference="camera_depth">
         <sensor name="depth_camera" type="depth_camera">
-            <pose relative_to='${namespace}/camera_depth'>0 0 0 0 0 0</pose>
+            <pose relative_to='camera_depth'>0 0 0 0 0 0</pose>
             <always_on>0</always_on>
             <update_rate>30</update_rate>
             <camera>
-                <optical_frame_id>${namespace}/camera_depth</optical_frame_id>
+                <optical_frame_id>camera_depth</optical_frame_id>
                 <horizontal_fov>1.019272</horizontal_fov> <!-- 58.4° -->
                 <image>
@@ -59,11 +59,11 @@
     </gazebo>
     <!--RGB Camera Astra Pro-->
-    <gazebo reference="${namespace}/camera_rgb">
+    <gazebo reference="camera_rgb">
         <sensor name="rgb_camera" type="camera">
-            <pose relative_to='${namespace}/camera_rgb'>0 0 0 0 0 0</pose>
+            <pose relative_to='camera_rgb'>0 0 0 0 0 0</pose>
             <always_on>0</always_on>
             <update_rate>30</update_rate>
             <camera>
-                <optical_frame_id>${namespace}/camera_rgb</optical_frame_id>
+                <optical_frame_id>camera_rgb</optical_frame_id>
                 <horizontal_fov>1.101303</horizontal_fov> <!-- 63.1° -->
                 <image>

File: src/helmoro_description/urdf/sensors/rplidar.urdf.xacro (robot description, xacro)
@@ -1,10 +1,10 @@
 <?xml version="1.1"?>
 <robot xmlns:xacro="http://ros.org/wiki/xacro">
-<xacro:macro name="rplidar" params="name namespace parent_link *origin">
+<xacro:macro name="rplidar" params="name parent_link *origin">
     <xacro:include filename="$(find helmoro_description)/urdf/utils.urdf.xacro"/>
-    <xacro:property name="joint_name" value="${namespace}/${name}_joint"/>
-    <xacro:property name="link_name" value="${namespace}/${name}"/>
+    <xacro:property name="joint_name" value="${name}_joint"/>
+    <xacro:property name="link_name" value="${name}"/>
     <joint name="${joint_name}" type="fixed">
-        <parent link="${namespace}/${parent_link}"/>
+        <parent link="${parent_link}"/>
         <child link="${link_name}"/>
         <xacro:insert_block name="origin"/>
